Commit message: fix:minor fix and change color of nexus

File: description/urdf/sml_nexus.gazebo.xacro (robot description, xacro)
@@ -41,5 +41,5 @@
   </gazebo>
   <gazebo reference="nexus_body">
-    <material>Gazebo/Yellow</material>
+    <material>Gazebo/Purple</material>
   </gazebo>
   <gazebo reference="left_sensor">

File: description/urdf/sml_nexus.xacro (robot description, xacro)
@@ -4,5 +4,5 @@
   <xacro:property name="wheel_radius" value="0.050" />
   <xacro:property name="wheel_width" value="0.0505" />
-  <material name="yellow"><color rgba="0.8 0.8 0.0 1.0" /></material>
+  <material name="yellow"><color rgba="1. 0.80 0.83 1.0" /></material>
   <material name="black"><color rgba="0.15 0.15 0.15 1.0" /></material>
   <material name="dark_grey"><color rgba="0.2 0.2 0.2 1.0" /></material>
